File: Sampling scope/Sampling scope.kicad_sch (KiCad schematic)
At the start: 0 parts

Commit message: add ldo schematic
Parts:
- added D1: SZESD8472MUT5G, SZESD8472MUT5G, symbol SamacSys_Parts:SZESD8472MUT5G
- added IC1: Si53360-B-GT, SamacSys_Parts:SOP65P640X120-16N, symbol SamacSys_Parts:Si53360-B-GT
- added IC2: LMK00304SQ, QFN50P500X500X80-33N, symbol SamacSys_Parts:LMK00304SQ
- added IC3: ADF4351BCPZ-RL7, QFN50P500X500X80-33N-D, symbol SamacSys_Parts:ADF4351BCPZ-RL7
- added IC4: MC100EP195FA, QFP80P900X900X160-32N, symbol SamacSys_Parts:MC100EP195FA
- added IC5: ADCMP582BCPZ-R2, QFN50P300X300X80-17N-D, symbol SamacSys_Parts:ADCMP582BCPZ-R2
- added IC6: TLV3601DBVR, SOT95P280X145-5N, symbol SamacSys_Parts:TLV3601DBVR
- added IC7: LTC2642IDD-16#PBF, SON50P300X300X80-11N-D, symbol SamacSys_Parts:LTC2642IDD-16#PBF
- added IC9: EP4CE6E22C8N, QFP50P2200X2200X165-145N, symbol SamacSys_Parts:EP4CE6E22C8N
- added J1: CH1, symbol Connector:Conn_Coaxial
- added J2: Trigger, symbol Connector:Conn_Coaxial
- added J3: REF_in, symbol Connector:Conn_Coaxial
- added J4: REF_out, symbol Connector:Conn_Coaxial
- added J5: GEN_out, symbol Connector:Conn_Coaxial
- added U1: NUCLEO144-H743ZI, Module:ST_Morpho_Connector_144_STLink, symbol MCU_Module:NUCLEO144-H743ZI
- added Y1: MV267, Oscillator:Oscillator_OCXO_Morion_MV267, symbol Oscillator:MV267
Connections:
- new net GND: J1.2 (Ext), J2.2 (Ext), J3.2 (Ext), J4.2 (Ext), J5.2 (Ext)
Other:
- added sheet Clock_distribution (Clock_distribution.kicad_sch)
- added sheet FPGA&MCU (FPGA&MCU.kicad_sch)
- added sheet Power (Power.kicad_sch)
- added sheet Sampler&Trigger (Sampler&Trigger.kicad_sch)
- note added: "CLK mux"
- note added: "DAC"
- note added: "Delay line"
- note added: "PLL"
- note added: "RF Synth"
- note added: "RF comp"
